File: electronics/DNC/modules/STM32F405.kicad_sch (KiCad schematic)
At the start: 32 parts

Commit message: Se reemplazó la hoja del IMU por la de sensores y se agregó la hoja de indicadores
- Nueva hoja Sensores: IMU BMI270 (SPI1) y barómetro BMP581 (I2C1 propio, jumper BARO_ADDR).
- Nueva hoja Indicadores: buzzer piezo CPT-12123 con FDV303N y LEDs de estado en PB4/PB5.
- Se eliminó la hoja IMU.
- MicroSD por SDIO de 4 bits con filtro TPD6F002 y TVS ESD5Z3.3 en VDD.
- PMS: AP2112K en 3V3_SYS y LP5907 + ferrita en 3V3_SEN.
- Motores movidos a PA0-PA3 (TIM5) para liberar el SDIO.
- Arquitectura.drawio actualizado a la arquitectura v1 (ELRS por UART, sin OLED).
- Se agregó docs/RESUMEN_PROYECTO_DNC.md con decisiones y pendientes.

Co-Authored-By: Claude Opus 5.5 <noreply@anthropic.com>
Parts:
- C? (x10): VOLTAGE 16V -> (none)
- FB?: CURRENT 350mA -> (none); PROVIDER LCSC -> (none); Price 0.0039 -> (none)
- U?: PROVIDER Mouser -> (none); Price 12.51 -> (none)
Connections:
- net CURR_SENSE: now also U?.27 (PB1)
- net VBAT_SENSE: now also U?.26 (PB0)
- net MTR1: now reaches U?.14 (PA0)
- net MTR2: now reaches U?.15 (PA1)
- net MTR3: now reaches U?.16 (PA2)
- net MTR4: now reaches U?.17 (PA3)
- net CSB: now reaches U?.20 (PA4)
- net SCK: now reaches U?.21 (PA5)
- net MISO: now reaches U?.22 (PA6)
- net MOSI: now reaches U?.23 (PA7)
- net INT1: now reaches U?.24 (PC4)
- net INT: now reaches U?.25 (PC5)
- net BUZZER: now reaches U?.41 (PA8)
- net DAT2: now reaches U?.51 (PC10)
- net DAT3: now reaches U?.52 (PC11)
- net CLK: now reaches U?.53 (PC12)
- net CMD: now reaches U?.54 (PD2)
- net LED_ERROR: now reaches U?.56 (PB4)
- net LED_STATUS: now reaches U?.57 (PB5)
- net SCL: now reaches U?.61 (PB8)
- net SDA: now reaches U?.62 (PB9)
- net MOTOR_1: no longer names the net of U?.37 (PC6)
- net MOTOR_2: no longer names the net of U?.38 (PC7)
- net MOTOR_3 renamed DAT0
- net MOTOR_4 renamed DAT1
- no-connect marks 34 -> 17
