File: electronics/DNC/modules/USB_POWER_IN.kicad_sch (KiCad schematic)
At the start: 6 parts

Commit message: Se reemplazó la hoja del IMU por la de sensores y se agregó la hoja de indicadores
- Nueva hoja Sensores: IMU BMI270 (SPI1) y barómetro BMP581 (I2C1 propio, jumper BARO_ADDR).
- Nueva hoja Indicadores: buzzer piezo CPT-12123 con FDV303N y LEDs de estado en PB4/PB5.
- Se eliminó la hoja IMU.
- MicroSD por SDIO de 4 bits con filtro TPD6F002 y TVS ESD5Z3.3 en VDD.
- PMS: AP2112K en 3V3_SYS y LP5907 + ferrita en 3V3_SEN.
- Motores movidos a PA0-PA3 (TIM5) para liberar el SDIO.
- Arquitectura.drawio actualizado a la arquitectura v1 (ELRS por UART, sin OLED).
- Se agregó docs/RESUMEN_PROYECTO_DNC.md con decisiones y pendientes.

Co-Authored-By: Claude Opus 5.5 <noreply@anthropic.com>
Parts:
- added D?: B5819W, symbol Device:D_Schottky_Filled
- FB?: LCSC Part C62708 -> (none); Mfr. Part CBM160808U121T -> (none); Price 0.0038 -> (none)
Connections:
- net VBUS_FILTER: now also D?.2 (A)
- new net 5V_SYS: D?.1 (K)
