File: electronics/DNC/modules/Indicadores.kicad_sch (KiCad schematic)
At the start: 10 parts

Commit message: Se enlazó el TPS54331 a la librería SJ (SJ_Power:TPS54331DDA)
- PMS: el TPS54331 pasa de DC-DC_Converter (own_symbols) a SJ_Power:TPS54331DDA.
  Netlist verificado: todas las redes iguales; el pad térmico (pin 9, ahora PAD) sigue en GND.
- Indicadores y raíz: cambios menores de KiCad (referencias sin anotar).

Co-Authored-By: Claude Opus 5.5 <noreply@anthropic.com>
Parts:
- renumbered D2 to D?, D1 to D?, R1 to R?
Changed lines of the file:
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@@
 		(dnp no)
 		(fields_autoplaced yes)
-		(property "Reference" "D2"
+		(property "Reference" "D?"
 			(at 191.77 99.3774 90)
 			(show_name no)
@@
 			(project "DNC"
 				(path "/abee636e-ad3a-4ba4-b95f-d0cf4a6d3d85/16b7fe8e-042e-4230-94b6-bdf3f83dd8c6"
-					(reference "D2")
+					(reference "D?")
 					(unit 1)
 				)
@@
 		(dnp no)
 		(fields_autoplaced yes)
-		(property "Reference" "R1"
+		(property "Reference" "R?"
 			(at 190.5 109.2199 0)
 			(show_name no)
@@
 			(project "DNC"
 				(path "/abee636e-ad3a-4ba4-b95f-d0cf4a6d3d85/16b7fe8e-042e-4230-94b6-bdf3f83dd8c6"
-					(reference "R1")
+					(reference "R?")
 					(unit 1)
 				)
@@
 		(dnp no)
 		(fields_autoplaced yes)
-		(property "Reference" "D1"
+		(property "Reference" "D?"
 			(at 191.77 66.3574 90)
 			(show_name no)
@@
 			(project "DNC"
 				(path "/abee636e-ad3a-4ba4-b95f-d0cf4a6d3d85/16b7fe8e-042e-4230-94b6-bdf3f83dd8c6"
-					(reference "D1")
+					(reference "D?")
 					(unit 1)
 				)
